File: kicad/modbus.sch (KiCad schematic (older format))
At the start: 20 parts, among them J1 Modbus, J16 Conn_01x03, J17 Conn_01x02, J18 Conn_01x02, J19 Conn_01x02, U8 SN65HVD11

Commit message: V0.1 Tapeout
Changed lines of the file:
@@
 EESchema Schematic File Version 2
-LIBS:rpi-hot-water-controller-rescue
 LIBS:power
 LIBS:device
@@
 LIBS:contrib
 LIBS:valves
-LIBS:import
-LIBS:import2
 LIBS:rpi-hot-water-controller-cache
 EELAYER 25 0
@@
 encoding utf-8
 Sheet 3 3
-Title ""
-Date ""
-Rev ""
-Comp ""
+Title "RPI Hot water controller"
+Date "2018-10-12"
+Rev "0.1"
+Comp "github.com/greenenergyprojects"
 Comment1 ""
 Comment2 ""
@@
 U 1 1 5BB6C6ED
 P 4800 2600
-F 0 "C16" V 4650 2500 50  0000 L CNN
+F 0 "C16" V 4650 2400 50  0000 L CNN
 F 1 "100n" V 4650 2650 50  0000 L CNN
 F 2 "Capacitors_SMD:C_1206_HandSoldering" H 4800 2600 50  0001 C CNN
@@
 $EndComp
 $Comp
-L GND #PWR087
+L GND #PWR089
 U 1 1 5BB6CF96
 P 5200 2700
-F 0 "#PWR087" H 5200 2450 50  0001 C CNN
+F 0 "#PWR089" H 5200 2450 50  0001 C CNN
 F 1 "GND" H 5200 2550 50  0000 C CNN
 F 2 "" H 5200 2700 50  0001 C CNN
@@
 $EndComp
 $Comp
-L +3V3 #PWR088
+L +3V3 #PWR090
 U 1 1 5BB6CF9C
 P 6600 1900
-F 0 "#PWR088" H 6600 1750 50  0001 C CNN
+F 0 "#PWR090" H 6600 1750 50  0001 C CNN
 F 1 "+3V3" H 6600 2040 50  0000 C CNN
 F 2 "" H 6600 1900 50  0001 C CNN
@@
 $EndComp
 $Comp
-L GND #PWR089
+L GND #PWR091
 U 1 1 5BB6D5DC
 P 7200 3400
-F 0 "#PWR089" H 7200 3150 50  0001 C CNN
+F 0 "#PWR091" H 7200 3150 50  0001 C CNN
 F 1 "GND" H 7200 3250 50  0000 C CNN
 F 2 "" H 7200 3400 50  0001 C CNN
@@
 $EndComp
 $Comp
-L +3V3 #PWR090
+L +3V3 #PWR092
 U 1 1 5BB6DABD
 P 4500 2300
-F 0 "#PWR090" H 4500 2150 50  0001 C CNN
+F 0 "#PWR092" H 4500 2150 50  0001 C CNN
 F 1 "+3V3" H 4500 2440 50  0000 C CNN
 F 2 "" H 4500 2300 50  0001 C CNN
@@
 $EndComp
 $Comp
-L +3V3 #PWR091
+L +3V3 #PWR093
 U 1 1 5BB6E094
 P 3000 2100
-F 0 "#PWR091" H 3000 1950 50  0001 C CNN
+F 0 "#PWR093" H 3000 1950 50  0001 C CNN
 F 1 "+3V3" H 3000 2240 50  0000 C CNN
 F 2 "" H 3000 2100 50  0001 C CNN
@@
 $EndComp
 $Comp
-L GND #PWR092
+L GND #PWR094
 U 1 1 5BB6E0DB
 P 4500 4100
-F 0 "#PWR092" H 4500 3850 50  0001 C CNN
+F 0 "#PWR094" H 4500 3850 50  0001 C CNN
 F 1 "GND" H 4500 3950 50  0000 C CNN
 F 2 "" H 4500 4100 50  0001 C CNN
@@
 $EndComp
 $Comp
-L GND #PWR093
+L GND #PWR095
 U 1 1 5BB6E122
 P 3800 4200
-F 0 "#PWR093" H 3800 3950 50  0001 C CNN
+F 0 "#PWR095" H 3800 3950 50  0001 C CNN
 F 1 "GND" H 3800 4050 50  0000 C CNN
 F 2 "" H 3800 4200 50  0001 C CNN
@@
 $EndComp
 $Comp
-L +3V3 #PWR094
+L +3V3 #PWR096
 U 1 1 5BB6E169
 P 3700 2500
-F 0 "#PWR094" H 3700 2350 50  0001 C CNN
+F 0 "#PWR096" H 3700 2350 50  0001 C CNN
 F 1 "+3V3" H 3700 2640 50  0000 C CNN
 F 2 "" H 3700 2500 50  0001 C CNN
@@
 RO
 $Comp
-L GND #PWR095
+L GND #PWR097
 U 1 1 5BB6F675
 P 6600 4700
-F 0 "#PWR095" H 6600 4450 50  0001 C CNN
+F 0 "#PWR097" H 6600 4450 50  0001 C CNN
 F 1 "GND" H 6600 4550 50  0000 C CNN
 F 2 "" H 6600 4700 50  0001 C CNN
