File: kicad/rpi-hot-water-controller.kicad_pcb (KiCad board)
At the start: 4 copper layers, 84.2 x 86.3 mm, 156 parts, among them J1 Modbus, J10 PT1000-2, J11 4-20mA, J12 PRJ_USB_MINI, J13 Atmega-ISP-6, J14 Conn_01x02, J15 Conn_01x04, J16 Conn_01x03, J17 Conn_01x02, J18 Conn_01x02, J19 Conn_01x02, J2 SSR1, J20 PRJ_Conn_01x03, J21 Drill-1, J22 Drill-2, J23 Conn_01x04, J24 TEST, J3 SSR2, J4 SSR4, J5 SSR5, J6 Screw_Terminal_01x03, J7 SENSOR-SUPPLY, J8 SENSOR-IN, J9 PT1000-1, K1 G3MB-202P, K2 G3MB-202P, K3 G3MB-202P, K4 G3MB-202P, P1 PRJ_Raspberry_Pi_2+, Q1 BSS138, Q2 BSS138, Q3 BSS138, Q4 BSS138, Q5 BSS138, Q6 BSS138, SW1 SW_Push, SW2 SW On/Off, U1 PRJ-UC-ATMEGA324P-20AU, U2 CH340G, U3 HLK-5M05, U4 PRJ_LM336M-2.5, U5 PRJ-supply-5VtoPM12V_ebay-253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, U6 LM358, U7 LM358, U8 SN65HVD11, X1 EXT1, X2 EXT2, X3 EXT3, X4 EXT4, Y1 12MHz, Y2 12MHz

Commit message: V0.1 Tapeout
Parts:
- removed the B4 at (179.5, 108.9)
- added B6: SOLDERBRDIGE-2, Project:SOLDER-JUMPER_1-WAY, F.Cu at (114.6, 109.7)
- added D19: green, LEDs:LED_0805_HandSoldering, F.Cu at (122.7, 67.7)
- added J25: Conn_01x03, Pin_Headers:Pin_Header_Straight_1x03_Pitch2.54mm, F.Cu at (184.2, 107.3)
- added R62: 680R, Resistors_SMD:R_1206_HandSoldering, B.Cu at (122.7, 76.2)
- B1: footprint Project:SOLDER-JUMPER_2-WAY -> Pin_Headers:Pin_Header_Straight_1x03_Pitch2.54mm
- C1: footprint Capacitors_SMD:C_1206_HandSoldering -> Capacitors_SMD:C_0805_HandSoldering; moved to B.Cu
- D14: moved to B.Cu
- D15, D16: footprint Diodes_SMD:D_0805 -> LEDs:LED_0805_HandSoldering
- R17: value 8k2 -> 6k8
- R20: value 6k8 -> 2k7
- R21: value 1k -> 470R
- R24: value 12k -> 15k
- R31, R33, R46, R48: value 1k5 -> 680R
- R40, R41: value 560 -> 680R
- R51: value 470 -> 680R
- SW1: footprint Buttons_Switches_SMD:SW_SPST_FSMSM -> Project:PRJ_SW_SPST_FSMSM
- moved C1 9.02 mm to (105.0, 110.5), turned to 180 degrees
- moved B1 3.82 mm to (120.1, 97.5), turned to 180 degrees
- moved D6 2.69 mm to (116.7, 107.1)
- moved D14 2.67 mm to (183.1, 114.6)
- moved C16 2.54 mm to (112.0, 118.4)
- moved C2 1.91 mm to (116.5, 106.4)
- moved SW1 1.91 mm to (126.6, 95.8)
- moved J12 1.65 mm to (110.1, 110.5)
- moved U2 1.46 mm to (116.8, 112.5)
- moved U8 1.40 mm to (117.0, 114.6)
- moved R15 1.27 mm to (126.2, 109.0)
- moved C4 0.77 mm to (125.0, 93.9), turned to 180 degrees
- moved R5 0.76 mm to (125.0, 91.7)
- moved Y2 0.57 mm to (124.0, 112.0)
- moved R4 0.51 mm to (125.7, 98.6)
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- renumbered B6 to B4
Connections:
- C2 pad 2: Net-(C2-Pad2) -> +3V3
- U2 pad 16: Net-(C2-Pad2) -> +3V3
- U2 pad 4: Net-(C2-Pad2) -> +3V3
Routing:
- net +3V3: track 98.6 -> 116.5 mm, vias 20 -> 22
- net GND: track 235.0 -> 250.9 mm, vias 33 -> 30
- net Net-(B1-Pad3): track 16.6 -> 30.4 mm
- net +5V: track 98.8 -> 111.2 mm
- net Net-(B1-Pad2): track 15.4 -> 3.30 mm, vias 1 -> 0
- net Net-(C2-Pad2): track 10.1 -> 0.00 mm
- net Net-(D19-Pad1): track 0.00 -> 7.99 mm, vias 0 -> 1
- net Net-(B6-Pad2): track 6.45 -> 12.8 mm
- net Net-(D14-Pad2): track 10.5 -> 15.1 mm
- net /~RST~: track 37.7 -> 41.7 mm
- net /UC-TxD0: track 41.0 -> 37.7 mm
- net /Modbus/RO: track 48.5 -> 51.4 mm
- net /InputOutput/PWM: track 113.1 -> 110.2 mm
- net /D+: track 22.5 -> 24.8 mm
- net Net-(J18-Pad1): track 14.1 -> 15.8 mm
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Other:
- board text added: "(C) github.com/greenenergyprojects"
- board text added: "(PB4)"
- board text added: "(PC6)"
- board text added: "5V"
- board text added: "A"
- board text added: "B"
- board text added: "B2: 2.5V<->AREF B3: AGND<->GND"
- board text added: "RESET from"
- board text added: "rpi-hot-water-controller V0.1 / sx"
- board text removed: "B2: 2.5V<->AREF"
- board text removed: "B3: AGND<->GND"
- board text removed: "LED PC6"
- board text removed: "PB4"
