File: kicad/rpi-hot-water-controller.sch (KiCad schematic (older format))
At the start: 59 parts, among them J12 PRJ_USB_MINI, J13 Atmega-ISP-6, J14 Conn_01x02, J20 PRJ_Conn_01x03, J21 Drill-1, J22 Drill-2, J23 Conn_01x04, J24 TEST, J6 Screw_Terminal_01x03, P1 PRJ_Raspberry_Pi_2+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

Commit message: V0.1 Tapeout
Parts:
- removed B4: SOLDERBRDIGE-2, Project:SOLDER-JUMPER_1-WAY, symbol SOLDERBRDIGE-2
- added B6: SOLDERBRDIGE-2, Project:SOLDER-JUMPER_1-WAY, symbol SOLDERBRDIGE-2
- added D19: green, LEDs:LED_0805_HandSoldering, symbol LED
- added J25: Conn_01x03, Pin_Headers:Pin_Header_Straight_1x03_Pitch2.54mm, symbol Conn_01x03
- added R62: 680R, Resistors_SMD:R_1206_HandSoldering, symbol R
- B1: footprint Project:SOLDER-JUMPER_2-WAY -> Pin_Headers:Pin_Header_Straight_1x03_Pitch2.54mm
- C1: footprint Capacitors_SMD:C_1206_HandSoldering -> Capacitors_SMD:C_0805_HandSoldering
- D16: footprint Diodes_SMD:D_0805 -> LEDs:LED_0805_HandSoldering
- SW1: footprint Buttons_Switches_SMD:SW_SPST_FSMSM -> Project:PRJ_SW_SPST_FSMSM
- renumbered B6 to B4
Connections:
- net +3V3: now also C2.2, U2.16 (VCC), U2.4 (V3), D19.2 (A)
- net +5V: now also B6.1 (G1), J25.2 (Pin_2)
- net GND: now also J25.1 (Pin_1), R62.1
- net at D14.2 (A), U3.2 (+5V): now also J25.3 (Pin_3)
- net at C1.1, D6.2 (A), J12.1 (VBUS): now also B6.2 (G2)
- new net: D19.1 (K), R62.2
Other:
- note removed: "Check!!"
- moved on the sheet: C1
