File: kicad/io.sch (KiCad schematic (older format))
At the start: 77 parts, among them J10 PT1000-2, J11 4-20mA, J15 Conn_01x04, J2 SSR1, J3 SSR2, J4 SSR4, J5 SSR5, J7 SENSOR-SUPPLY, J8 SENSOR-IN, J9 PT1000-1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

Commit message: V0.1 Tapeout
Parts:
- D15: footprint Diodes_SMD:D_0805 -> LEDs:LED_0805_HandSoldering
- R17: value 8k2 -> 6k8
- R20: value 6k8 -> 2k7
- R21: value 1k -> 470R
- R24: value 12k -> 15k
- R31, R33, R46, R48: value 1k5 -> 680R
- R40, R41: value 560 -> 680R
- R51: value 470 -> 680R
Other:
- note added: "For µC-VREF=1.0V (B2 open):\nR17=8K2, R20=6K8, R21=1K, R24=12K\nRV1: Trim RV1 to PT1000-1=0.51V when\nR on J9 is 1K2"
- note added: "For µC-VREF=2.5V (B2 closed):\nR17=6K8, R20=2K7, R21=470R, R24=15K\nRV1: Trim RV1 to PT1000-1=1.35V when\nR on J9 is 1K2"
- note added: "Values for\nµC-VREF=1.0V (B2 open)"
- note added: "Values for\nµC-VREF=2.5V (B2 closed)"
- note removed: "Trim 1000 Ohm on J? to\n60mV ouput voltage"

Commit message: test finished for pcb release V0.1
Parts:
- J4: value SSR4 -> SSR3
- J5: value SSR5 -> SSR4
Changed lines of the file:
@@
 P 10500 4300
 F 0 "J4" H 10500 4100 50  0000 C CNN
-F 1 "SSR4" H 10700 4250 50  0000 C CNN
+F 1 "SSR3" H 10700 4250 50  0000 C CNN
 F 2 "Project:Terminalblock-2x-5,08mm_ebay-273426629807" H 10500 4300 50  0001 C CNN
 F 3 "" H 10500 4300 50  0001 C CNN
@@
 P 10500 5700
 F 0 "J5" H 10500 5500 50  0000 C CNN
-F 1 "SSR5" H 10700 5650 50  0000 C CNN
+F 1 "SSR4" H 10700 5650 50  0000 C CNN
 F 2 "Project:Terminalblock-2x-5,08mm_ebay-273426629807" H 10500 5700 50  0001 C CNN
 F 3 "" H 10500 5700 50  0001 C CNN

Commit message: ...
Other:
- note added: "Maximum VGS\nat least 12V!"
Changed lines of the file:
@@
 Text Notes 2650 1150 0    39   ~ 0
 Values for\nµC-VREF=2.5V (B2 closed)
+Text Notes 10400 2300 0    60   ~ 0
+Maximum VGS\nat least 12V!
 $EndSCHEMATC
